File: NPulse_v2/FSR.kicad_sch (KiCad schematic)
At the start: 111 parts, among them J14 Conn_01x02_Pin, J15 Conn_01x02_Pin, J16 Conn_01x02_Pin, J17 Conn_01x02_Pin, J18 Conn_01x02_Pin, J19 Conn_01x02_Pin, Q1 PMOS, Q2 PMOS, Q3 PMOS, Q4 PMOS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

Commit message: Version 3 - motor driver updated, FSR updated
Parts:
- added Q10, Q11, Q12, Q13, Q7, Q8, Q9: PNP, symbol Simulation_SPICE:PNP
- added R58, R61, R62, R63, R79, R80, R81, R82: R, symbol Device:R
- U19, U30, U32, U33, U34, U35: footprint Package_TO_SOT_SMD:SOT-353_SC-70-5 -> (none)
Connections:
- net +3.3V: now also R61.2, R62.2, R63.2, R79.2, R80.2, R81.2, R82.2
- net GND: now also R58.1
- net at J18.1 (Pin_1), R39.1: now also Q11.1 (C); no longer Q5.3 (S)
- net at J16.1 (Pin_1), R31.1: now also Q9.1 (C); no longer Q3.3 (S)
- net at J17.1 (Pin_1), R35.1: now also Q10.1 (C); no longer Q4.3 (S)
- net at J19.1 (Pin_1), R43.1: now also Q12.1 (C); no longer Q6.3 (S)
- net at J15.1 (Pin_1), R27.1: now also Q8.1 (C); no longer Q2.3 (S)
- net at J14.1 (Pin_1), R23.1: now also Q13.1 (C); no longer Q1.3 (S)
- new net: Q13.3 (E), R82.1
- new net: Q10.2 (B), Q11.2 (B), Q12.2 (B), Q13.2 (B), Q7.1 (C), Q7.2 (B), Q8.2 (B), Q9.2 (B), R58.2
- new net: Q11.3 (E), R80.1
- new net: Q7.3 (E), R61.1
- new net: Q8.3 (E), R62.1
- new net: Q9.3 (E), R63.1
- new net: Q12.3 (E), R81.1
- new net: Q10.3 (E), R79.1
Other:
- note added: "1.6mV par degrée"
- note added: "1V au bord de R61 environ 1k"
- note added: "3.9 ou 4.7k"
- note added: "5 - une jonction (=0.65) -> 4.35V Courant base négligeable donc R61 et R58 se répartissent 4.35V"
- note added: "faire un pont diviseur de tension et relié pour tout le monde et ajouté au milieu une 0.1uF au milieu à la masse"
- note removed: "https://www.electronique-et-informatique.fr/Digit/Digit_4TS2.php"
- note removed: "selon la place et les pins restantes sur le mcu : transistors pour faire un switch piloté et bypass le filtrage Sinon des jumpers mécaniques mais bon -> 12 jumpers"
- moved on the sheet: Q1, Q2, Q3, Q4, Q5, Q6, R20, R21, R22, R52, R53, R54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
