File: NPulse_v2/motor_driver2.kicad_sch (KiCad schematic)
At the start: 48 parts, among them J10 Screw_Terminal_01x02, J11 Screw_Terminal_01x02, J12 Screw_Terminal_01x02, J13 Screw_Terminal_01x02, U11 74HC00, U12 74HC00, U13 DRV8212P, U14 DRV8212P, U15 74HC00, U16 74HC00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

Commit message: Version 3 - motor driver updated, FSR updated
Parts:
- U13, U14, U17, U18: footprint Package_SON:WSON-8-1EP_2x2mm_P0.5mm_EP0.9x1.6mm_ThermalVias -> (none)
Changed lines of the file:
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@@
 			)
 		)
-		(property "Footprint" "Package_SON:WSON-8-1EP_2x2mm_P0.5mm_EP0.9x1.6mm_ThermalVias"
+		(property "Footprint" ""
 			(at 95.25 76.2 0)
 			(effects
@@
 			)
 		)
-		(property "Footprint" "Package_SON:WSON-8-1EP_2x2mm_P0.5mm_EP0.9x1.6mm_ThermalVias"
+		(property "Footprint" ""
 			(at 231.14 76.2 0)
 			(effects
@@
 			)
 		)
-		(property "Footprint" "Package_SON:WSON-8-1EP_2x2mm_P0.5mm_EP0.9x1.6mm_ThermalVias"
+		(property "Footprint" ""
 			(at 231.14 143.51 0)
 			(effects
@@
 			)
 		)
-		(property "Footprint" "Package_SON:WSON-8-1EP_2x2mm_P0.5mm_EP0.9x1.6mm_ThermalVias"
+		(property "Footprint" ""
 			(at 96.52 143.51 0)
 			(effects
