File: NPulse_v2/test.kicad_sch (KiCad schematic)
At the start: 15 parts, among them IC2 DRV8220DSGR, J20 Conn_01x05_Pin, J3 Screw_Terminal_01x02, U39 TXB0102DCT, U42 74HC00

Commit message: Version 3 - motor driver updated, FSR updated
Parts:
- C118: value C -> 100nF
- IC2: footprint SON50P200X200X80-9N -> (none)
- R59: value R -> 1k
- R60: value R -> 2 ou 1
- U39: footprint Package_SO:TSSOP-8_3x3mm_P0.65mm -> (none)
- U42: value 74HC00 -> 74LVC00
Connections:
- net +3.3V: now also IC2.8 (NSLEEP), U42.12, U42.13
- net GND: no longer C114.2, C115.2, C117.2, C119.1, IC2.7 (MODE)
- net pin4: now reaches IC2.4 (GND), R59.2, R60.1
- net pin4: now also C114.2, C115.2, C117.2, C119.1, IC2.7 (MODE)
Other:
- note added: "C119, C114, C115, C117 à la pin 4 pour éviter les rebouclages de courant Mode aussi à pin 4"
- note added: "Package_DFN_QFN:DHVQFN-14-1EP_2.5x3mm_P0.5mm_EP1x1.5mm"
- note added: "Thermal pad au terminal de la pin 4"
- note added: "Un bornier de 16 plots, méchaniquement c'est mieux pas de 2.54mm, (rq: plus épais qu'un bornier à vis pour le même pas)"
- note added: "faible"
- note added: "grande par rapport à R60"
- moved on the sheet: C118, J3, R59, R60
