File: NPulse_v3/FSR.kicad_sch (KiCad schematic)
At the start: 15 parts, among them J12 Conn_01x02_Pin, J14 Conn_01x02_Pin, J15 Conn_01x02_Pin, J16 Conn_01x02_Pin, J17 Conn_01x02_Pin

Commit message: Version 4
Parts:
- removed C69, C70, C71, C72: C, symbol Device:C
- removed J12, J14, J15, J16, J17: Conn_01x02_Pin, symbol Connector:Conn_01x02_Pin
- removed R25, R26, R27, R28: R, symbol Device:R
- added C21, C22, C23, C24: 100nF, Capacitor_SMD:C_0402_1005Metric, symbol Device:C
- added J5: Conn_01x10_Pin, Bornier10:1725737, symbol Connector:Conn_01x10_Pin
- added R17, R18, R19, R20: 1k, Resistor_SMD:R_0402_1005Metric, symbol Device:R
- C20: renamed from C67; value C -> 100nF; footprint (none) -> Capacitor_SMD:C_0402_1005Metric
- R16: renamed from R23; value R -> 1k; footprint (none) -> Resistor_SMD:R_0402_1005Metric
Connections:
- net +3.3V: now also R17.1, R18.1, R19.1, R20.1
- net GND: now also C21.1, C22.1, C23.1, C24.1, J5.10 (Pin_10), J5.2 (Pin_2), J5.4 (Pin_4), J5.6 (Pin_6), J5.8 (Pin_8)
- net FSR_1 renamed FSR1
- net FSR1: now also J5.1 (Pin_1)
- new net FSR2: C22.2, J5.3 (Pin_3), R18.2
- new net FSR3: C24.2, J5.5 (Pin_5), R20.2
- new net FSR4: C21.2, J5.7 (Pin_7), R17.2
- new net FSR5: C23.2, J5.9 (Pin_9), R19.2
Other:
- moved on the sheet: C20, R16
