File: NPulse_v3/NPulse_v3.kicad_sch (KiCad schematic)
At the start: 32 parts, among them IC2 TXU0202QDCURQ1, J1 Conn_01x04_Pin, J2 Conn_01x04_Pin, J3 Conn_01x06_Pin, SW1 SW_Push, SW2 SW_SPDT, U1 STM32G484METx, Y1 16MHz

Commit message: Version 4
Parts:
- removed IC2: TXU0202QDCURQ1, symbol TXU0202QDCURQ1:TXU0202QDCURQ1
- added C11: 1uF, Capacitor_SMD:C_0402_1005Metric, symbol Device:C
- added C12, C17: 100nF, Capacitor_SMD:C_0402_1005Metric, symbol Device:C
- added H1, H2, H3, H4: MountingHole, MountingHole:MountingHole_2.2mm_M2, symbol Mechanical:MountingHole
- added IC1: TXU0202QDCURQ1, TXU:SOP50P310X90-8N, symbol new_components:TXU0202QDCURQ1
- added J1: Conn_01x04_Pin, Connector_PinHeader_2.54mm:PinHeader_1x04_P2.54mm_Vertical, symbol Connector:Conn_01x04_Pin
- added Q1: PMOS, PMOS:SOT95P240X120-3N, symbol Simulation_SPICE:PMOS
- added Q2: NMOS, NMOS:SOT95P240X120-3N, symbol Simulation_SPICE:NMOS
- added R1, R2, R3, R4, R5: 1k, Resistor_SMD:R_0402_1005Metric, symbol Device:R
- added R10, R6, R7: 10k, Resistor_SMD:R_0402_1005Metric, symbol Device:R
- added R8: 47k, Resistor_SMD:R_0402_1005Metric, symbol Device:R
- C1: footprint (none) -> Capacitor_SMD:C_0805_2012Metric
- C10, C2, C3, C4, C5, C6, C7, C8, C9: footprint (none) -> Capacitor_SMD:C_0402_1005Metric
- C13: renamed from C11; footprint (none) -> Capacitor_SMD:C_0402_1005Metric
- C14: renamed from C13; footprint (none) -> Capacitor_SMD:C_0402_1005Metric
- C15: renamed from C14; footprint (none) -> Capacitor_SMD:C_0402_1005Metric
- C16: renamed from C15; footprint (none) -> Capacitor_SMD:C_0402_1005Metric
- C18: renamed from C17; footprint (none) -> Capacitor_SMD:C_0402_1005Metric
- C19: renamed from C18; footprint (none) -> Capacitor_SMD:C_0402_1005Metric
- D1: footprint (none) -> Photodiode:SOD6439X180N
- FB1: footprint (none) -> Inductor_SMD:L_0402_1005Metric
- J2: renamed from J1; footprint (none) -> Connector_PinHeader_2.54mm:PinHeader_1x04_P2.54mm_Vertical
- J3: footprint (none) -> Connector_PinHeader_2.54mm:PinHeader_1x06_P2.54mm_Vertical
- J4: renamed from J2; footprint (none) -> Connector_PinHeader_2.54mm:PinHeader_1x04_P2.54mm_Vertical
- R11: renamed from R4; footprint (none) -> Resistor_SMD:R_0402_1005Metric
- R12: renamed from R5; footprint (none) -> Resistor_SMD:R_0402_1005Metric
- R13: renamed from R6; footprint (none) -> Resistor_SMD:R_0805_2012Metric
- R14: renamed from R3; footprint (none) -> Resistor_SMD:R_0402_1005Metric
- R15: renamed from R2; footprint (none) -> Resistor_SMD:R_0402_1005Metric
- R9: renamed from R1; footprint (none) -> Resistor_SMD:R_0402_1005Metric
- SW1: footprint (none) -> Button_Switch_THT:SW_PUSH_6mm
- SW2: footprint (none) -> Button_Switch_SMD:SW_SPDT_PCM12
- U1: footprint (none) -> Package_QFP:LQFP-80_12x12mm_P0.5mm
- Y1: footprint (none) -> Crystal:Crystal_SMD_3225-4Pin_3.2x2.5mm
Connections:
- net DIR_5 is gone; now on net EMG_RX: U1.71 (PD2)
- net ENC_6 is gone; now on net EMG_TX: U1.68 (PC12)
- net I_6 is gone; now on net LED: U1.13 (PA1)
- net +3.3V: now also IC1.3 (VCCA)
- net +3.3VA: now also R1.1
- net GND: now also C11.2, C12.2, C17.2, IC1.2 (GND), Q2.3 (S), R10.2
- net LED: no longer U1.56 (PA8)
- net RX: now also IC1.8 (B1Y); no longer R12.1, U1.67 (PC11)
- net TX: now also IC1.1 (B2); no longer U1.66 (PC10)
- net VCCB: now also IC1.6 (OE), IC1.7 (VCCB)
- net EMG_RX: now reaches R14.2
- net EMG_TX: now reaches R15.2
- net NSS: now reaches U1.18 (PA4)
- net NSS: now also R2.1
- net SCK: now reaches U1.19 (PA5)
- net SCK: now also R3.1
- net DIR8: now reaches U1.2 (PC13)
- net MISO: now reaches U1.20 (PA6)
- net MISO: now also R4.1
- net MOSI: now reaches U1.21 (PA7)
- net MOSI: now also R5.1
- net ENC3_S1: now reaches U1.25 (PB1)
- net at U1.28 (VREF+): now also C11.1, C12.1, R1.2
- net ENC1_S2: now reaches U1.3 (PC14)
- net I3: now reaches U1.33 (PE10)
- net I1: now reaches U1.34 (PE11)
- net I4: now reaches U1.35 (PE12)
- net PWM4: now reaches U1.36 (PE13)
- net DIR4: now reaches U1.37 (PE14)
- net ENC5_S2: now reaches U1.38 (PE15)
- net ENC1_S1: now reaches U1.4 (PC15)
- net ENC6_S2: now reaches U1.60 (PA12)
- net ENC7_S1: now reaches U1.73 (PB4)
- net ENC7_S2: now reaches U1.74 (PB5)
- net PWM7: now reaches U1.75 (PB6)
- net DIR7: now reaches U1.76 (PB7)
- net DIR_1 renamed PWM8
- net DIR_2: no longer names the net of U1.39 (PB10)
- net DIR_3 renamed MesOn
- net MesOn: now also Q2.2 (G)
- net DIR_4 renamed NSLEEP
- net DIR_6 renamed I2
- net DIR_7 renamed I7
- net DIR_8 renamed I8
- net ENC_1 renamed ENC8_S1
- net ENC_2 renamed ENC8_S2
- net ENC_3 renamed I5
- net ENC_4 renamed ENC2_S2
- net ENC_5: no longer names the net of U1.26 (PB2)
- net ENC_7 renamed DIR3
- net ENC_8 renamed PWM3
- net FSR_1 renamed FSR1
- net FSR_2 renamed FSR2
- net FSR_3 renamed FSR3
- net FSR_4 renamed FSR4
- net FSR_5 renamed FSR5
- net I_1 renamed DIR1
- net I_2 renamed PWM1
- net I_3 renamed ENC4_S1
- net I_4 renamed ENC4_S2
- net I_5 renamed AD_Vbat
- net AD_Vbat: now also C17.1, R10.1, R8.1
- net I_7 renamed ENC2_S1
- net I_8 renamed ENC3_S2
- net PWM_1 renamed ENC5_S1
- net PWM_2 renamed ENC6_S1
- net PWM_3 renamed DIR2
- net PWM_4 renamed PWM2
- net PWM_5 renamed DIR5
- net PWM_6 renamed PWM5
- net PWM_7 renamed DIR6
- net PWM_8 renamed PWM6
- new net: Q2.1 (D), R7.2
- new net: Q1.1 (D), R8.2
- new net: Q1.2 (G), R6.2, R7.1
- new net: J1.4 (Pin_4), R2.2
- new net: J1.1 (Pin_1), R5.2
- new net: J1.2 (Pin_2), R4.2
- new net: J1.3 (Pin_3), R3.2
- new net I6: U1.56 (PA8)
- new net RX_UART4: IC1.4 (A2Y), R12.1, U1.67 (PC11)
- new net TX_UART4: IC1.5 (A1), U1.66 (PC10)
- new net Vbat: Q1.3 (S), R6.1
- no-connect marks 2 -> 5
Other:
- note added: "ADC pins"
- note added: "ADC1_IN1 : PA0 (2) ADC1_IN2 : PA1 (2) ADC1_IN3 : PA2 ADC1_IN4 : PA3 ADC1_IN5 : PB14 (4) ADC1_IN6 : PC0 (2) ADC1_IN7 : PC1 (2) ADC1_IN8 : PC2 (2) ADC1_IN9 : PC3 (2) ADC1_IN10 : PF0 ADC1_IN11 : PB12 (4) ADC1_IN12 : PB1 (3) ADC1_IN14 : PB11 (2) ADC1_IN15 : PB0 (3)"
- note added: "ADC2_IN1 : PA0 (1) ADC2_IN2 : PA1 (1) ADC2_IN3 : PA6 ADC2_IN4 : PA7 ADC2_IN5 : PC4 ADC2_IN6 : PC0 (1) ADC2_IN7 : PC1 (1) ADC2_IN8 : PC2 (1) ADC2_IN9 : PC3 (1) ADC2_IN10 : PF1 ADC2_IN11 : PC5 ADC2_IN12 : PB2 ADC2_IN13 : PA5 ADC2_IN14 : PB11 (1) ADC2_IN15 : PB15 (4) ADC2_IN17 : PA4"
- note added: "ADC3_IN1 : PB1 (1) ADC3_IN2 : PE9 ADC3_IN3 : PE13 ADC3_IN4 : PE7 ADC3_IN5 : PB13 ADC3_IN6 : PE8 (4, 5) ADC3_IN7 : PD10 (4, 5) ADC3_IN12 : PB0 (1) ADC3_IN14 : PE10 (4, 5) ADC3_IN15 : PE11 (4, 5) ADC3_IN16 : PE12 (4, 5)"
- note added: "ADC4_IN1 : PE14 ADC4_IN2 : PE15 ADC4_IN3 : PB12 (1) ADC4_IN4 : PB14 (1) ADC4_IN5 : PB15 (2) ADC4_IN6 : PE8 (3, 5) ADC4_IN7 : PD10 (3, 5) ADC4_IN12 : PD8 (5) ADC4_IN13 : PD9 (5) ADC4_IN14 : PE10 (3, 5) ADC4_IN15 : PE11 (3, 5) ADC4_IN16 : PE12 (3, 5)"
- note added: "ADC5_IN1 : PA8 ADC5_IN2 : PA9 ADC5_IN6 : PE8 (3, 4) ADC5_IN7 : PD10 (3, 4) ADC5_IN12 : PD8 (4) ADC5_IN13 : PD9 (4) ADC5_IN14 : PE10 (3, 4) ADC5_IN15 : PE11 (3, 4) ADC5_IN16 : PE12 (3, 4)"
- note added: "NMOS : VSS138 PMOS : VSS84"
- note added: "TIM2 (32 bits): CH1 (PA0, PA5, PA15), CH2 (PA1, PB3) TIM5 (32 bits) : CH1 (PA0, PB2), CH2 (PA1, PC12) TIM3 (16 bits): CH1 (PA6, PC6, PB4), CH2 (PA4, PA7, PC7, PB5) TIM4 (16 bits): CH1 (PA11, PB6), CH2 (PA12, PB7)"
- note added: "TIMER 1 : CH1 (PC0, PE9, PA8), CH2 (PC1, PE11, PA9), CH3 (PC2, PE13, PA10), CH4 (PC3, PE14, PA11) TIMER 8 : CH1 (PC6, PA15, PB6), CH2 (PC7, PA14, PB8), CH3 (PC8, PB9), CH4 (PC9, PD1)"
- note added: "UART Protocol (to EMG) UART5"
- note added: "UART Protocol (to computer) UART4"
- note added: "enc 1, 3, 4, 5 soft"
- note added: "eventually 3 wires (without VCC)"
- note removed: "TIM2 (32 bits): CH1 (PA0, PA5, PA15), CH2 (PA1, PB3), CH3 (PA2, PA9, PB10), CH4 (PA3, PA10, PB11) (max 4) TIM5 (32 bits) : CH1 (PA0, PB2), CH2 (PA1, PC12), CH3 (PA2, PE8), CH4 (PA3, PE9) (max 4) TIM3 (16 bits) TIM4 (16 bits)"
- note removed: "TIMER 1 : PC0, PC1, PC2, PC3, PA8, PA9, PA10, PA11 (max 4) TIMER 8 : PB6, PB7, PB8, PB9, PC6, PC7, PC8, PC9 (max 4)"
- note removed: "UART Protocol (to EMG Board)"
- note removed: "UART Protocol (to computer)"
- note removed: "prévoir un SPI pour communiquer avec l'IMU"
- moved on the sheet: C13, C14, C15, C16, C18, D1, J2, J3, J4, R13, R14, R15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
