File: NPulse_v3/motor_driver.kicad_sch (KiCad schematic)
At the start: 104 parts, among them IC10 DRV8220DSGR, IC3 DRV8220DSGR, IC4 DRV8220DSGR, IC5 DRV8220DSGR, IC6 DRV8220DSGR, IC7 DRV8220DSGR, IC8 DRV8220DSGR, IC9 DRV8220DSGR, J10 Screw_Terminal_01x02, J11 Screw_Terminal_01x02, J4 Screw_Terminal_01x02, J5 Screw_Terminal_01x02, J6 Screw_Terminal_01x02, J7 Screw_Terminal_01x02, J8 Screw_Terminal_01x02, J9 Screw_Terminal_01x02, U2 74LVC00, U3 74LVC00, U4 74LVC00, U5 74LVC00, U6 74LVC00, U7 74LVC00, U8 74LVC00, U9 74LVC00

Commit message: Version 4
Parts:
- removed C19, C21: 100nF, symbol Device:C
- removed C20, C22: 10uF, symbol Device:C
- removed C23, C24: C, symbol Device:C
- removed IC10, IC3, IC4, IC5, IC6, IC7, IC8, IC9: DRV8220DSGR, symbol DRV8220DSGR:DRV8220DSGR
- removed J10, J11, J4, J5, J6, J7, J8, J9: Screw_Terminal_01x02, symbol Connector:Screw_Terminal_01x02
- removed R10, R13, R14, R17, R18, R9: 2 ou 1, symbol Device:R
- removed R11, R12, R15, R16, R19, R20, R7, R8: 1k, symbol Device:R
- removed U2, U3, U4, U5, U6, U7, U8, U9: 74LVC00, symbol 74xx:74HC00
- added C67, C68, C71, C72: 100nF, Capacitor_SMD:C_0402_1005Metric, symbol Device:C
- added C69, C70: 10uF, Capacitor_SMD:C_0805_2012Metric, symbol Device:C
- added IC2, IC3, IC4, IC5, IC6, IC7, IC8, IC9: DRV8220DSGR, DRV8220DSGR:WSON8_DSG_TEX, symbol new_components:DRV8220DSGR
- added J10, J7, J8, J9: 1725753, bornier12:1725753, symbol bornier:1725753
- added R23, R24, R27, R28, R31, R32, R35, R36: 1, Resistor_SMD:R_1020_2550Metric, symbol Device:R
- added R25, R26, R29, R30, R33, R34: 1k, Resistor_SMD:R_0402_1005Metric, symbol Device:R
- added U2, U3, U4, U5, U6, U7, U8, U9: 74HC02, Package_DFN_QFN:DHVQFN-14-1EP_2.5x3mm_P0.5mm_EP1x1.5mm, symbol 74xx:74HC02
- C25, C31, C37, C43, C49, C55, C61: footprint (none) -> Capacitor_SMD:C_0402_1005Metric
- C26, C29, C30, C33, C38, C41, C42, C45, C50, C53, C54, C57, C62, C65, C66: value 100nF -> 10uF; footprint (none) -> Capacitor_SMD:C_0805_2012Metric
- C27, C35, C36, C39, C47, C48, C51, C59, C60, C63: value C -> 100nF; footprint (none) -> Capacitor_SMD:C_0402_1005Metric
- C28, C40, C52, C64: value C -> 10uF; footprint (none) -> Capacitor_SMD:C_0805_2012Metric
- C32, C44, C56: value 10uF -> 100nF; footprint (none) -> Capacitor_SMD:C_0402_1005Metric
- C34, C46, C58: footprint (none) -> Capacitor_SMD:C_0805_2012Metric
- L1, L10, L11, L12, L13, L14, L15, L16, L2, L3, L4, L5, L6, L7, L8, L9: value L -> 10uH; footprint (none) -> 10uH_bob:LQH5BPB100MT0L
- R21, R22: value 2 ou 1 -> 1k; footprint (none) -> Resistor_SMD:R_0402_1005Metric
Connections:
- net I_1 is gone; now on an unnamed net: C29.1
- net I_2 is gone; now on an unnamed net: C41.1
- net I_3 is gone; now on an unnamed net: C53.1
- net I_4 is gone; now on an unnamed net: C65.1
- net I_5 is gone; now on an unnamed net: C30.1
- net I_6 is gone; now on an unnamed net: C42.1
- net I_7 is gone; now on an unnamed net: C54.1
- net I_8 is gone; now on an unnamed net: C66.1
- net +12V: now also C25.2, C26.1, C27.2, C28.1, C37.2, C38.1, C39.2, C40.1, C49.2, C50.1, C51.2, C52.1, C61.2, C62.1, C63.2, C64.1, IC2.1 (VM), IC3.1 (VM), IC4.1 (VM), IC5.1 (VM), IC6.1 (VM), IC7.1 (VM), IC8.1 (VM), IC9.1 (VM); no longer C31.2, C32.1, C33.2, C34.1, C43.2, C44.1, C45.2, C46.1, C55.2, C56.1, C57.2, C58.1
- net +3.3V: now also C31.1, C32.1, C43.1, C44.1, C55.1, C56.1, C67.1, C68.1, U2.14 (VCC), U3.14 (VCC), U4.14 (VCC), U5.14 (VCC), U6.14 (VCC), U7.14 (VCC), U8.14 (VCC), U9.14 (VCC); no longer C25.1, C26.1, C37.1, C38.1, C49.1, C50.1, C61.1, C62.1
- net GND: now also C31.2, C32.2, C35.2, C36.2, C43.2, C44.2, C47.2, C48.2, C55.2, C56.2, C59.2, C60.2, C67.2, C68.2, C71.2, C72.2, J10.2, J10.8, J7.2, J7.8, J8.2, J8.8, J9.2, J9.8, R23.2, R24.2, R27.2, R28.2, R31.2, R32.2, R35.2, R36.2, U2.7 (GND), U3.7 (GND), U4.7 (GND), U5.7 (GND), U6.7 (GND), U7.7 (GND), U8.7 (GND), U9.7 (GND); no longer C25.2, C26.2, C29.2, C30.2, C37.2, C38.2, C41.2, C42.2, C49.2, C50.2, C53.2, C54.2, C61.2, C62.2, C65.2, C66.2, R21.2, R22.2
- net at L16.2: now also C70.1, J10.12; no longer C64.1
- net at L10.2: now also J10.1; no longer C48.1
- net at L13.2: now also J9.7; no longer C59.1
- net at L15.2: now also C69.1, J9.12; no longer C63.1
- net at L6.1: now also IC5.2 (OUT1)
- net at L8.1: now also IC5.3 (OUT2)
- net at L2.1: now also IC3.2 (OUT1)
- net at L4.1: now also IC3.3 (OUT2)
- net at L5.1: now also IC4.2 (OUT1)
- net at L5.2: now also J7.7; no longer C35.1
- net at L3.2: now also C33.1, J7.6; no longer C27.1
- net at L1.2: now also J7.1
- net at L12.2: now also C58.1, J10.6; no longer C52.1
- net at L9.2: now also J9.1; no longer C47.1
- net at L9.1: now also IC6.2 (OUT1)
- net at L6.2: now also J8.7; no longer C36.1
- net at L11.1: now also IC6.3 (OUT2)
- net at L11.2: now also C57.1, J9.6; no longer C51.1
- net at L14.1: now also IC9.2 (OUT1)
- net at L14.2: now also J10.7; no longer C60.1
- net at L3.1: now also IC2.3 (OUT2)
- net at L2.2: now also J8.1
- net at L7.1: now also IC4.3 (OUT2)
- net at L7.2: now also C45.1, J7.12; no longer C39.1
- net at L1.1: now also IC2.2 (OUT1)
- net at L15.1: now also IC8.3 (OUT2)
- net at L4.2: now also C34.1, J8.6; no longer C28.1
- net at L10.1: now also IC7.2 (OUT1)
- net at L12.1: now also IC7.3 (OUT2)
- net at L16.1: now also IC9.3 (OUT2)
- net at L8.2: now also C46.1, J8.12; no longer C40.1
- net at L13.1: now also IC8.2 (OUT1)
- removed net pin4: C27.2, C28.2, C31.1, C32.2, C33.1, C34.2, C35.2, C36.2, C39.2, C40.2, C43.1, C44.2, C45.1, C46.2, C47.2, C48.2, C51.2, C52.2, C55.1, C56.2, C57.1, C58.2, C59.2, C60.2, C63.2, C64.2, R21.1, R22.1
- new net: U2.3, U2.4
- new net: U9.10, U9.11, U9.2
- new net: U9.3, U9.4
- new net: U3.3, U3.4
- new net: U4.10, U4.11, U4.2
- new net: U4.3, U4.4
- new net: U8.3, U8.4
- new net: U2.10, U2.11, U2.2
- new net: U5.10, U5.11, U5.2
- new net: U3.10, U3.11, U3.2
- new net: U7.3, U7.4
- new net: U5.3, U5.4
- new net: U6.10, U6.11, U6.2
- new net: U7.10, U7.11, U7.2
- new net: U8.10, U8.11, U8.2
- new net: U6.3, U6.4
- new net +4.5V: J10.11, J10.5, J7.11, J7.5, J8.11, J8.5, J9.11, J9.5
- new net DIR1: U2.12, U2.5, U2.6
- new net DIR2: U4.12, U4.5, U4.6
- new net DIR3: U6.12, U6.5, U6.6
- new net DIR4: U8.12, U8.5, U8.6
- new net DIR5: U3.12, U3.5, U3.6
- new net DIR6: U5.12, U5.5, U5.6
- new net DIR7: U7.12, U7.5, U7.6
- new net DIR8: U9.12, U9.5, U9.6
- new net ENC1_S1: J7.3
- new net ENC1_S2: J7.4
- new net ENC2_S1: J7.9
- new net ENC2_S2: J7.10
- new net ENC3_S1: J9.3
- new net ENC3_S2: J9.4
- new net ENC4_S1: J9.9
- new net ENC4_S2: J9.10
- new net ENC5_S1: J8.3
- new net ENC5_S2: J8.4
- new net ENC6_S1: J8.9
- new net ENC6_S2: J8.10
- new net ENC7_S1: J10.3
- new net ENC7_S2: J10.4
- new net ENC8_S1: J10.9
- new net ENC8_S2: J10.10
- new net I1: C35.1, R21.1
- new net I2: C47.1, R25.1
- new net I3: C59.1, R29.1
- new net I4: C71.1, R33.1
- new net I5: C36.1, R22.1
- new net I6: C48.1, R26.1
- new net I7: C60.1, R30.1
- new net I8: C72.1, R34.1
- new net NSLEEP: IC2.8 (NSLEEP), IC3.8 (NSLEEP), IC4.8 (NSLEEP), IC5.8 (NSLEEP), IC6.8 (NSLEEP), IC7.8 (NSLEEP), IC8.8 (NSLEEP), IC9.8 (NSLEEP)
- new net OUT1_1: IC2.6 (IN1/PH), U2.13
- new net OUT1_2: IC2.5 (IN2/EN), U2.1
- new net OUT2_1: IC4.6 (IN1/PH), U4.13
- new net OUT2_2: IC4.5 (IN2/EN), U4.1
- new net OUT3_1: IC6.6 (IN1/PH), U6.13
- new net OUT3_2: IC6.5 (IN2/EN), U6.1
- new net OUT4_1: IC8.6 (IN1/PH), U8.13
- new net OUT4_2: IC8.5 (IN2/EN), U8.1
- new net OUT5_1: IC3.6 (IN1/PH), U3.13
- new net OUT5_2: IC3.5 (IN2/EN), U3.1
- new net OUT6_1: IC5.6 (IN1/PH), U5.13
- new net OUT6_2: IC5.5 (IN2/EN), U5.1
- new net OUT7_1: IC7.6 (IN1/PH), U7.13
- new net OUT7_2: IC7.5 (IN2/EN), U7.1
- new net OUT8_1: IC9.6 (IN1/PH), U9.13
- new net OUT8_2: IC9.5 (IN2/EN), U9.1
- new net PWM1: U2.8, U2.9
- new net PWM2: U4.8, U4.9
- new net PWM3: U6.8, U6.9
- new net PWM4: U8.8, U8.9
- new net PWM5: U3.8, U3.9
- new net PWM6: U5.8, U5.9
- new net PWM7: U7.8, U7.9
- new net PWM8: U9.8, U9.9
- new net pin4_1: C25.1, C26.2, C29.2, C33.2, IC2.4 (GND), R21.2, R23.1
- new net pin4_2: C37.1, C38.2, C41.2, C45.2, IC4.4 (GND), R25.2, R27.1
- new net pin4_3: C49.1, C50.2, C53.2, C57.2, IC6.4 (GND), R29.2, R31.1
- new net pin4_4: C61.1, C62.2, C65.2, C69.2, IC8.4 (GND), R33.2, R35.1
- new net pin4_5: C27.1, C28.2, C30.2, C34.2, IC3.4 (GND), R22.2, R24.1
- new net pin4_6: C39.1, C40.2, C42.2, C46.2, IC5.4 (GND), R26.2, R28.1
- new net pin4_7: C51.1, C52.2, C54.2, C58.2, IC7.4 (GND), R30.2, R32.1
- new net pin4_8: C63.1, C64.2, C66.2, C70.2, IC9.4 (GND), R34.2, R36.1
Other:
- note added: "81-LQH5BPB100MT0L"
- note added: "C119, C114, C115, C117 à la pin 4 pour éviter les rebouclages de courant"
- note added: "Motor VCC Encoder GND Encoder Signal 1 Encoder Signal 2 Encoder VCC Motor GND"
- note added: "shunt"
- note removed: "C119, C114, C115, C117, Mode à la pin 4 pour éviter les rebouclages de courant"
- note removed: "faible"
