File: NPulse_v4/connecteur_v2/connecteur_v2.kicad_sch (KiCad schematic)
At the start: 26 parts, among them J1 Conn_01x02_Socket, J10 Conn_02x05_Odd_Even, J13 Conn_02x05_Odd_Even, J2 Conn_01x02_Socket, J23 Conn_01x01, J24 Conn_01x06_Socket, J25 Conn_01x06_Socket, J26 Conn_01x06_Socket, J27 Conn_01x01, J28 Conn_01x06_Socket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

Commit message: add text on hat board, generate gerbers
Parts:
- J6: footprint Connector_JST:JST_PH_B4B-PH-SM4-TB_1x04-1MP_P2.00mm_Vertical -> Connector_JST:JST_PH_B4B-PH-K_1x04_P2.00mm_Vertical
Changed lines of the file:
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@@
 			)
 		)
-		(property "Footprint" "Connector_JST:JST_PH_B4B-PH-SM4-TB_1x04-1MP_P2.00mm_Vertical"
+		(property "Footprint" "Connector_JST:JST_PH_B4B-PH-K_1x04_P2.00mm_Vertical"
 			(at 218.44 36.83 0)
 			(effects
